Commit message: model second ver

File: scara_description/urdf/scara_description.urdf (robot description, URDF)
Before this commit: robot scara_description, 8 links, 7 joints
Joints:
- joint joint1: limit lower=0 upper=252.45 effort=200 velocity=3 -> lower=-0.25245 upper=0 effort=200 velocity=3
- joint joint2: origin xyz=0 0 0 rpy=0 0 0 -> xyz=0.014 0.0935 0.1372 rpy=0 0 0
- joint joint3: limit lower=-1.34390352 upper=4.01425728 effort=200 velocity=3 -> lower=-1.3439 upper=4.0143 effort=200 velocity=3; origin xyz=0 0 0 rpy=0 0 0 -> xyz=0.215 0 0.0453999999999997 rpy=0 0 -1.5707963267949
- joint joint4: origin xyz=0 0 0 rpy=0 0 0 -> xyz=0 0.285 0.0416 rpy=0 0 -1.5707963267949
- joint joint5: axis 0 1 0 -> 0 0 -1; limit lower=0 upper=0.69813 effort=200 velocity=3 -> lower=-0.69813 upper=0 effort=200 velocity=3; origin xyz=0 0 0 rpy=0 0 0 -> xyz=0 -0.047 0.092 rpy=-1.5707963267949 0 0
- joint joint6: axis -1 0 0 -> 0 0 1; origin xyz=0 0 0 rpy=0 0 0 -> xyz=-0.0178499999999999 0 0.048 rpy=1.5707963267949 0 1.5707963267949
- joint joint7: axis 0 1 0 -> 0 0 1; limit lower=-1.57079633 upper=0.17453293 effort=200 velocity=3 -> lower=-1.5708 upper=0.17453 effort=200 velocity=3; origin xyz=0 0 0 rpy=0 0 0 -> xyz=0 0 -0.078405 rpy=1.5708 -1.5708 0

Commit message: model fifth ver

File: scara_description/urdf/scara_description.urdf (robot description, URDF)
Before this commit: robot scara_description, 8 links, 7 joints
Links:
- link link2: mass 0.58092 -> 0.580917463575827
- link link3: mass 0.30095 -> 0.300947531370299
- link link4: mass 0.16132 -> 0.161315962203164
- link link5: mass 0.15899 -> 0.158985625581691
- link link6: mass 0.071797 -> 0.0717968221721648
- link link7: mass 0.065589 -> 0.0655886884429779
Joints:
- joint joint3: origin xyz=0.215 0 0.0453999999999997 rpy=0 0 -1.5707963267949 -> xyz=0.215 0 0.0454 rpy=0 0 -1.5708
- joint joint4: origin xyz=0 0.285 0.0416 rpy=0 0 -1.5707963267949 -> xyz=0.0935 -0.229 -0.1826 rpy=0 0 1.5708
- joint joint5: origin xyz=0 -0.047 0.092 rpy=-1.5707963267949 0 0 -> xyz=0.514 0.1405 0.3162 rpy=-1.5708 0 3.1416
- joint joint6: origin xyz=-0.0178499999999999 0 0.048 rpy=1.5707963267949 0 1.5707963267949 -> xyz=-0.01785 0 0.048 rpy=1.5708 0 1.5708

Commit message: moveit config 1st, model 6th

File: scara_description/urdf/scara_description.urdf (robot description, URDF)
Before this commit: robot scara_description, 8 links, 7 joints
Links:
- link link2: mass 0.580917463575827 -> 0.58092
- link link3: mass 0.300947531370299 -> 0.30095
- link link4: mass 0.161315962203164 -> 0.16132
- link link5: mass 0.158985625581691 -> 0.15899
- link link6: mass 0.0717968221721648 -> 0.071797
- link link7: mass 0.0655886884429779 -> 0.065589
Joints:
- joint joint4: origin xyz=0.0935 -0.229 -0.1826 rpy=0 0 1.5708 -> xyz=0 0.285 0.0416 rpy=0 0 -1.5708
- joint joint5: origin xyz=0.514 0.1405 0.3162 rpy=-1.5708 0 3.1416 -> xyz=0 -0.047 0.092 rpy=-1.5708 0 0
- joint joint7: limit lower=-1.5708 upper=0.17453 effort=200 velocity=3 -> lower=-0.17453 upper=1.5708 effort=200 velocity=3

Commit message: moveit motion planning succeed

File: scara_description/urdf/scara_description.urdf (robot description, URDF)
Before this commit: robot scara_description, 8 links, 7 joints
Links:
- added link link8, mass 0.037459; collision mesh filename=package://scara_description/meshes/link8.STL; visual mesh filename=package://scara_description/meshes/link8.STL
- link base_link: mass 0.57218 -> None
- link link7: mass 0.065589 -> 0.02813
Joints:
- added joint joint8: type fixed, parent link7, child link8, origin xyz=0.0 0.0 0.0 rpy=0.0 0.0 0.0, axis 0.0 0.0 0.0
- joint joint1: axis 0 0 -1 -> 0.0 0.0 -1; origin xyz=0 0 0 rpy=0 0 0 -> xyz=0.0 0.0 0.0 rpy=0.0 0.0 0.0
- joint joint2: axis 0 0 1 -> 0.0 0.0 1.0; origin xyz=0.014 0.0935 0.1372 rpy=0 0 0 -> xyz=0.014 0.0935 0.1372 rpy=0.0 0.0 0.0
- joint joint3: axis 0 0 1 -> 0.0 0.0 1.0; origin xyz=0.215 0 0.0454 rpy=0 0 -1.5708 -> xyz=0.215 0 0.0454 rpy=0.0 0.0 -1.5708
- joint joint4: axis 0 0 1 -> 0.0 0.0 1.0; origin xyz=0 0.285 0.0416 rpy=0 0 -1.5708 -> xyz=0 0.285 0.0416 rpy=0.0 0.0 -1.5708
- joint joint5: axis 0 0 -1 -> 0.0 0.0 -1
- joint joint6: axis 0 0 1 -> 0.0 0.0 1.0
- joint joint7: axis 0 0 1 -> 0.0 0.0 1.0; limit lower=-0.17453 upper=1.5708 effort=200 velocity=3 -> lower=-1.5708 upper=0.17453 effort=200 velocity=3; origin xyz=0 0 -0.078405 rpy=1.5708 -1.5708 0 -> xyz=0.0 0.0 -0.078405 rpy=1.5708 -1.5708 0

Commit message: module bug fixed

File: scara_description/urdf/scara_description.urdf (robot description, URDF)
Before this commit: robot scara_description, 9 links, 8 joints
Links:
- link base_link: mass None -> 0.57217968365953
- link link1: mass 0.27253 -> 0.27252514896887
- link link2: mass 0.58092 -> 0.580917463575827
- link link3: mass 0.30095 -> 0.300947531370299
- link link4: mass 0.16132 -> 0.161315962203164
- link link5: mass 0.15899 -> 0.158985625581691
- link link6: mass 0.071797 -> 0.0717968221721647
- link link7: mass 0.02813 -> 0.0281299504553923
- link link8: mass 0.037459 -> 0.0374587379875856
Joints:
- joint joint1: axis 0.0 0.0 -1 -> 0 0 -1; origin xyz=0.0 0.0 0.0 rpy=0.0 0.0 0.0 -> xyz=0 0 0 rpy=0 0 0
- joint joint2: axis 0.0 0.0 1.0 -> 0 0 1; origin xyz=0.014 0.0935 0.1372 rpy=0.0 0.0 0.0 -> xyz=0.014 0.0935 0.1372 rpy=0 0 0
- joint joint3: axis 0.0 0.0 1.0 -> 0 0 1; origin xyz=0.215 0 0.0454 rpy=0.0 0.0 -1.5708 -> xyz=0.215 0 0.0453999999999997 rpy=0 0 -1.5707963267949
- joint joint4: axis 0.0 0.0 1.0 -> 0 0 1; origin xyz=0 0.285 0.0416 rpy=0.0 0.0 -1.5708 -> xyz=0 0.285 0.0416 rpy=0 0 -1.5707963267949
- joint joint5: axis 0.0 0.0 -1 -> 0 0 -1; origin xyz=0 -0.047 0.092 rpy=-1.5708 0 0 -> xyz=0 -0.047 0.092 rpy=-1.5707963267949 0 0
- joint joint6: axis 0.0 0.0 1.0 -> 0 0 1; origin xyz=-0.01785 0 0.048 rpy=1.5708 0 1.5708 -> xyz=-0.0178499999999999 0 0.048 rpy=1.5707963267949 0 1.5707963267949
- joint joint7: axis 0.0 0.0 1.0 -> 0 0 1; limit lower=-1.5708 upper=0.17453 effort=200 velocity=3 -> lower=-0.17453 upper=1.5708 effort=200 velocity=3; origin xyz=0.0 0.0 -0.078405 rpy=1.5708 -1.5708 0 -> xyz=0 0 -0.078405 rpy=1.5708 -1.5708 0
- joint joint8: axis 0.0 0.0 0.0 -> 0 0 0; origin xyz=0.0 0.0 0.0 rpy=0.0 0.0 0.0 -> xyz=0 0 0 rpy=0 0 0

Commit message: initial pose added, update joint limits

File: scara_description/urdf/scara_description.urdf (robot description, URDF)
Before this commit: robot scara_description, 9 links, 8 joints
Joints:
- joint joint3: limit lower=-1.3439 upper=4.0143 effort=200 velocity=3 -> lower=-2.618 upper=2.618 effort=200 velocity=3
- joint joint5: limit lower=-0.69813 upper=0 effort=200 velocity=3 -> lower=0.0 upper=0.69813 effort=200 velocity=3
- joint joint6: limit lower=-3.1416 upper=0 effort=200 velocity=3 -> lower=-1.5708 upper=1.5708 effort=200 velocity=3
